Commit message: Improves humanoid robot's locomotion
Adds a reward term to penalize feet getting too close together, preventing awkward gaits.

Updates the mass of the ankle roll link to improve stability.

Adds a MuJoCo XML file for improved simulation fidelity.

File: source/robot_lab/robot_lab/assets/descriptions/urdf0924/urdf/urdf0924.urdf (robot description, URDF)
Before this commit: robot urdf0924, 28 links, 27 joints
Links:
- link right_ankle_roll_link: mass 0.19236845 -> 1.1728
